File: hardware/BDSM.sch (KiCad schematic (older format))
At the start: 5 parts, among them J1 614105150721, SW1 \"ON/OFF\"

Commit message: Fix ESP32 powering errors
Other:
- note removed: "Watch Dog!!!!"
Changed lines of the file:
@@
 Wire Wire Line
 	3600 4250 3600 4350
-Text Notes 7300 6850 0    79   ~ 0
-Watch Dog!!!!
 $Comp
 L Device:LED_Small LD2
