File: hardware/ESP32.sch (KiCad schematic (older format))
At the start: 40 parts, among them Q1 BC847, Q2 BC847, Q3 BSS138, Q4 BSS138, Q5 BSS138, U5 USBLC6-2SC6, U6 CH340G, U7 ESP32-WROOM-32D, Y1 12MHz

Commit message: Fix ESP32 powering errors
Parts:
- Q1, Q2: value BC847 -> SS8050; PartNumber BC847.215 -> SS8050
- U5: symbol Power_Protection:USBLC6-2SC6 -> BDSM-rescue:USBLC6-2SC6-Power_Protection
- U7: symbol ESP32:ESP32 -> BDSM-rescue:ESP32-ESP32
- Y1: PartNumber ABM3-8.000MHZ-D2Y-T -> ABM3-12.000MHZ-D2Y-T
Connections:
- net +3V3: now also C15.1, C16.1, C18.1, U6.16 (VCC), U6.4 (V3)
- net VBUS: no longer C15.1, C16.1, U6.16 (VCC)
- net MCU-PWR-CNTRL: no longer names the net of U7.27 (GPIO16)
Other:
- note added: "Replace Q1,Q2 to SS8050."
Changed lines of the file:
@@
 	2500 1650 2500 1750
 $Comp
-L ESP32:ESP32 U?
+L BDSM-rescue:ESP32-ESP32 U?
 U 1 1 5EFD7B8A
 P 4650 1850
@@
 $EndComp
 Wire Wire Line
-	4500 5450 4500 5000
+	4500 5450 4500 5150
 Wire Wire Line
 	3000 5000 3000 5100
@@
 F 2 "PatternLibs:ABM3" H 3250 6450 50  0001 C CNN
 F 3 "~" H 3250 6450 50  0001 C CNN
-F 4 "ABM3-8.000MHZ-D2Y-T" H 3250 6450 50  0001 C CNN "PartNumber"
+F 4 "ABM3-12.000MHZ-D2Y-T" H 3250 6450 50  0001 C CNN "PartNumber"
 	1    3250 6450
 	1    0    0    -1
@@
 AR Path="/5EFBEA8E/5F08D7BC" Ref="Q1"  Part="1"
 F 0 "Q1" H 6391 6096 50  0000 L CNN
-F 1 "BC847" H 6391 6005 50  0000 L CNN
+F 1 "SS8050" H 6391 6005 50  0000 L CNN
 F 2 "Package_TO_SOT_SMD:SOT-23" H 6400 5975 50  0001 L CIN
 F 3 "http://www.infineon.com/dgdl/Infineon-BC847SERIES_BC848SERIES_BC849SERIES_BC850SERIES-DS-v01_01-en.pdf?fileId=db3a304314dca389011541d4630a1657" H 6200 6050 50  0001 L CNN
-F 4 "BC847.215" H 6200 6050 50  0001 C CNN "PartNumber"
+F 4 "SS8050" H 6200 6050 50  0001 C CNN "PartNumber"
 	1    6200 6050
 	1    0    0    -1
@@
 AR Path="/5EFBEA8E/5F08D7C9" Ref="Q2"  Part="1"
 F 0 "Q2" H 6391 6796 50  0000 L CNN
-F 1 "BC847" H 6391 6705 50  0000 L CNN
+F 1 "SS8050" H 6391 6705 50  0000 L CNN
 F 2 "Package_TO_SOT_SMD:SOT-23" H 6400 6675 50  0001 L CIN
 F 3 "http://www.infineon.com/dgdl/Infineon-BC847SERIES_BC848SERIES_BC849SERIES_BC850SERIES-DS-v01_01-en.pdf?fileId=db3a304314dca389011541d4630a1657" H 6200 6750 50  0001 L CNN
-F 4 "BC847.215" H 6200 6750 50  0001 C CNN "PartNumber"
+F 4 "SS8050" H 6200 6750 50  0001 C CNN "PartNumber"
 	1    6200 6750
 	1    0    0    1
@@
 Text Label 5500 5650 0    50   ~ 0
 RXD0
-Connection ~ 3000 5000
 Text Label 3150 5950 0    50   ~ 0
 D+
@@
 Wire Wire Line
 	1500 5000 2600 5000
-Text HLabel 6600 3050 2    50   Output ~ 0
-MCU-PWR-CNTRL
 Text HLabel 1500 5500 0    50   BiDi ~ 0
 USB-D+
@@
 $EndComp
 $Comp
-L Power_Protection:USBLC6-2SC6 U5
+L BDSM-rescue:USBLC6-2SC6-Power_Protection U5
 U 1 1 5EFC47AB
 P 2000 6000
@@
 Wire Wire Line
 	2600 6000 2600 5000
-Connection ~ 2600 5000
-Wire Wire Line
-	2600 5000 3000 5000
 $Comp
 L power:GNDA #PWR?
@@
 Wire Wire Line
 	4500 2950 4700 2950
-Wire Wire Line
-	6600 3050 6400 3050
 $Comp
 L Device:CP1_Small C?
@@
 Text Label 5150 4050 3    50   ~ 0
 SPI_MOSI
+Text Notes 5200 7100 0    50   ~ 0
+Replace Q1,Q2 to SS8050.
+$Comp
+L power:+3.3V #PWR?
+U 1 1 5F689D2C
+P 3000 4800
+AR Path="/5EF9D67C/5F689D2C" Ref="#PWR?"  Part="1"
+AR Path="/5EFBEA8E/5F689D2C" Ref="#PWR0102"  Part="1"
+F 0 "#PWR0102" H 3000 4650 50  0001 C CNN
+F 1 "+3.3V" H 3015 4973 50  0000 C CNN
+F 2 "" H 3000 4800 50  0001 C CNN
+F 3 "" H 3000 4800 50  0001 C CNN
+	1    3000 4800
+	1    0    0    -1
+$EndComp
+Wire Wire Line
+	3000 4800 3000 5000
+Connection ~ 3000 5000
+Wire Wire Line
+	4400 5150 4500 5150
+Connection ~ 4400 5150
+Connection ~ 4500 5150
+Wire Wire Line
+	4500 5150 4500 5000
 $EndSCHEMATC
