File: hardware/Power.sch (KiCad schematic (older format))
At the start: 38 parts, among them U1 MAX16054AZT+T, U2 BQ24070, U3 TPS63001, U4 STC3100

Commit message: Fix ESP32 powering errors
Parts:
- removed TP3: MCU-PWR, TestPoint:TestPoint_Pad_1.0x1.0mm, symbol Connector:TestPoint_Alt
- U1: symbol Mainboard:MAX16054 -> BDSM-rescue:MAX16054-Mainboard
- U2: symbol Mainboard:BQ24070 -> BDSM-rescue:BQ24070-Mainboard
- U4: symbol Telemetry:STC3100 -> BDSM-rescue:STC3100-Telemetry
- XP1: symbol Mainboard:CONN-2M -> BDSM-rescue:CONN-2M-Mainboard
Connections:
- net MCU-PWR-CNTRL: no longer names the net of R2.2, U1.3 (CLEAR)
