File: hardware/SENSORS.sch (KiCad schematic (older format))
At the start: 14 parts, among them U8 MPU-6050, U9 MPU-9250

Commit message: Fix ESP32 powering errors
Parts:
- R32: value 10k -> DNP; PartNumber RC0603FR-0710KL -> DNP
- U9: value MPU-9250 -> DNP (MPU-9250 ); PartNumber MPU-9250 -> DNP
Changed lines of the file:
@@
 AR Path="/5EFBEEB7/5EFD21BC" Ref="U9"  Part="1"
 F 0 "U9" H 8100 4100 50  0000 C CNN
-F 1 "MPU-9250" H 8100 2500 50  0000 C CNN
+F 1 "DNP (MPU-9250 )" H 8100 2500 50  0000 C CNN
 F 2 "Sensor_Motion:InvenSense_QFN-24_3x3mm_P0.4mm" H 7800 2300 50  0001 C CNN
 F 3 "https://store.invensense.com/datasheets/invensense/MPU9250REV1.0.pdf" H 7800 3150 50  0001 C CNN
-F 4 "MPU-9250" H 7800 3300 50  0001 C CNN "PartNumber"
+F 4 "DNP" H 7800 3300 50  0001 C CNN "PartNumber"
 	1    7800 3300
 	1    0    0    -1
@@
 AR Path="/5EFBEEB7/5F031FCA" Ref="R32"  Part="1"
 F 0 "R32" H 6750 2050 50  0000 C CNN
-F 1 "10k" H 6750 2150 50  0000 C CNN
+F 1 "DNP" H 6750 2150 50  0000 C CNN
 F 2 "Resistor_SMD:R_0603_1608Metric" H 6900 2100 50  0001 C CNN
 F 3 "~" H 6900 2100 50  0001 C CNN
-F 4 "RC0603FR-0710KL" H 6900 2100 50  0001 C CNN "PartNumber"
+F 4 "DNP" H 6900 2100 50  0001 C CNN "PartNumber"
 	1    6900 2100
 	-1   0    0    1
